Commit message: gazebo launch

File: mechabot_ws/src/mechabot_description/urdf/mechabot_base.xacro (robot description, xacro)
@@ -3,6 +3,11 @@
     <link name="base_footprint"/>
     <link name="base_link">
-        <visual>
+        <inertial>
             <origin xyz="0.0 0.0 -0.0125" rpy="0.0 0.0 0.0"/>
+            <mass value="5.0"/>
+            <inertia ixx="0.1" ixy="0.0" ixz="0.0" iyy="0.1" iyz="0.0" izz="0.1"/>
+        </inertial>
+        <visual>
+            <origin xyz="0.0 0.0 -0.0125" rpy="0.0 0.0 0.0"/>
             <geometry>
                 <mesh filename="package://mechabot_description/meshes/mechabot_base_link.stl" scale="0.001 0.001 0.001"/>
@@ -12,4 +17,13 @@
             </material>
         </visual>
+        <collision>
+            <origin xyz="0.0 0.0 -0.0125" rpy="0.0 0.0 0.0"/>
+            <geometry>
+                <mesh filename="package://mechabot_description/meshes/mechabot_base_link.stl" scale="0.001 0.001 0.001"/>
+            </geometry>
+            <material name="grey">
+                <color rgba="0.8 0.8 0.8 1.0"/>
+            </material>
+        </collision>
     </link>
     <joint name="base_joint" type="fixed">
@@ -19,6 +33,11 @@
     </joint>
     <link name="right_wheel_link">
-        <visual>
+        <inertial>
             <origin xyz="0.0 0.0925 -0.034" rpy="0.0 0.0 0.0"/>
+            <mass value="0.5"/>
+            <inertia ixx="0.1" ixy="0.0" ixz="0.0" iyy="0.1" iyz="0.0" izz="0.1"/>
+        </inertial>
+        <visual>
+            <origin xyz="0.0 0.0925 -0.034" rpy="0.0 0.0 0.0"/>
             <geometry>
                 <mesh filename="package://mechabot_description/meshes/mechabot_right_wheel.stl" scale="0.001 0.001 0.001"/>
@@ -28,4 +47,13 @@
             </material>
         </visual>
+        <collision>
+            <origin xyz="0.0 0.0925 -0.034" rpy="0.0 0.0 0.0"/>
+            <geometry>
+                <mesh filename="package://mechabot_description/meshes/mechabot_right_wheel.stl" scale="0.001 0.001 0.001"/>
+            </geometry>
+            <material name="blue">
+                <color rgba="0.0 0.0 0.6 1.0"/>
+            </material>
+        </collision>
     </link>
     <joint name="right_wheel_joint" type="continuous">
@@ -36,6 +64,11 @@
     </joint>
     <link name="left_wheel_link">
-        <visual>
+        <inertial>
             <origin xyz="0.0 -0.0925 -0.034" rpy="0.0 0.0 0.0"/>
+            <mass value="0.5"/>
+            <inertia ixx="0.1" ixy="0.0" ixz="0.0" iyy="0.1" iyz="0.0" izz="0.1"/>
+        </inertial>
+        <visual>
+            <origin xyz="0.0 -0.0925 -0.034" rpy="0.0 0.0 0.0"/>
             <geometry>
                 <mesh filename="package://mechabot_description/meshes/mechabot_left_wheel.stl" scale="0.001 0.001 0.001"/>
@@ -45,4 +78,13 @@
             </material>
         </visual>
+        <collision>
+            <origin xyz="0.0 -0.0925 -0.034" rpy="0.0 0.0 0.0"/>
+            <geometry>
+                <mesh filename="package://mechabot_description/meshes/mechabot_left_wheel.stl" scale="0.001 0.001 0.001"/>
+            </geometry>
+            <material name="blue">
+                <color rgba="0.0 0.0 0.6 1.0"/>
+            </material>
+        </collision>
     </link>
     <joint name="left_wheel_joint" type="continuous">
@@ -53,6 +95,11 @@
     </joint>
     <link name="front_right_castor_link">
-        <visual>
+        <inertial>
             <origin xyz="-0.085 0.065 -0.021" rpy="0.0 0.0 0.0"/>
+            <mass value="0.2"/>
+            <inertia ixx="0.1" ixy="0.0" ixz="0.0" iyy="0.1" iyz="0.0" izz="0.1"/>
+        </inertial>
+        <visual>
+            <origin xyz="-0.085 0.065 -0.021" rpy="0.0 0.0 0.0"/>
             <geometry>
                 <mesh filename="package://mechabot_description/meshes/front_right_castor.stl" scale="0.001 0.001 0.001"/>
@@ -62,4 +109,13 @@
             </material>
         </visual>
+        <collision>
+            <origin xyz="-0.085 0.065 -0.021" rpy="0.0 0.0 0.0"/>
+            <geometry>
+                <mesh filename="package://mechabot_description/meshes/front_right_castor.stl" scale="0.001 0.001 0.001"/>
+            </geometry>
+            <material name="grey">
+                <color rgba="0.8 0.8 0.8 1.0"/>
+            </material>
+        </collision>
     </link>
     <joint name="front_right_castor_joint" type="fixed">
@@ -69,6 +125,11 @@
     </joint>
     <link name="front_left_castor_link">
-        <visual>
+        <inertial>
             <origin xyz="-0.085 -0.065 -0.021" rpy="0.0 0.0 0.0"/>
+            <mass value="0.2"/>
+            <inertia ixx="0.1" ixy="0.0" ixz="0.0" iyy="0.1" iyz="0.0" izz="0.1"/>
+        </inertial>
+        <visual>
+            <origin xyz="-0.085 -0.065 -0.021" rpy="0.0 0.0 0.0"/>
             <geometry>
                 <mesh filename="package://mechabot_description/meshes/front_left_castor.stl" scale="0.001 0.001 0.001"/>
@@ -78,4 +139,13 @@
             </material>
         </visual>
+        <collision>
+            <origin xyz="-0.085 -0.065 -0.021" rpy="0.0 0.0 0.0"/>
+            <geometry>
+                <mesh filename="package://mechabot_description/meshes/front_left_castor.stl" scale="0.001 0.001 0.001"/>
+            </geometry>
+            <material name="grey">
+                <color rgba="0.8 0.8 0.8 1.0"/>
+            </material>
+        </collision>
     </link>
     <joint name="front_left_castor_joint" type="fixed">
@@ -85,6 +155,11 @@
     </joint>
     <link name="rear_right_castor_link">
-        <visual>
+        <inertial>
             <origin xyz="0.085 0.065 -0.0205" rpy="0.0 0.0 0.0"/>
+            <mass value="0.2"/>
+            <inertia ixx="0.1" ixy="0.0" ixz="0.0" iyy="0.1" iyz="0.0" izz="0.1"/>
+        </inertial>
+        <visual>
+            <origin xyz="0.085 0.065 -0.0205" rpy="0.0 0.0 0.0"/>
             <geometry>
                 <mesh filename="package://mechabot_description/meshes/rear_right_castor.stl" scale="0.001 0.001 0.001"/>
@@ -94,4 +169,13 @@
             </material>
         </visual>
+        <collision>
+            <origin xyz="0.085 0.065 -0.0205" rpy="0.0 0.0 0.0"/>
+            <geometry>
+                <mesh filename="package://mechabot_description/meshes/rear_right_castor.stl" scale="0.001 0.001 0.001"/>
+            </geometry>
+            <material name="grey">
+                <color rgba="0.8 0.8 0.8 1.0"/>
+            </material>
+        </collision>
     </link>
     <joint name="rear_right_castor_joint" type="fixed">
@@ -101,6 +185,11 @@
     </joint>
     <link name="rear_left_castor_link">
-        <visual>
+        <inertial>
             <origin xyz="0.085 -0.065 -0.0205" rpy="0.0 0.0 0.0"/>
+            <mass value="0.2"/>
+            <inertia ixx="0.1" ixy="0.0" ixz="0.0" iyy="0.1" iyz="0.0" izz="0.1"/>
+        </inertial>
+        <visual>
+            <origin xyz="0.085 -0.065 -0.0205" rpy="0.0 0.0 0.0"/>
             <geometry>
                 <mesh filename="package://mechabot_description/meshes/rear_left_castor.stl" scale="0.001 0.001 0.001"/>
@@ -110,4 +199,13 @@
             </material>
         </visual>
+        <collision>
+            <origin xyz="0.085 -0.065 -0.0205" rpy="0.0 0.0 0.0"/>
+            <geometry>
+                <mesh filename="package://mechabot_description/meshes/rear_left_castor.stl" scale="0.001 0.001 0.001"/>
+            </geometry>
+            <material name="grey">
+                <color rgba="0.8 0.8 0.8 1.0"/>
+            </material>
+        </collision>
     </link>
     <joint name="rear_left_castor_joint" type="fixed">
@@ -117,4 +215,9 @@
     </joint>
     <link name="toplid_link">
+        <inertial>
+            <origin xyz="0.0 0.0 -0.1125" rpy="0.0 0.0 0.0"/>
+            <mass value="2.0"/>
+            <inertia ixx="0.1" ixy="0.0" ixz="0.0" iyy="0.1" iyz="0.0" izz="0.1"/>
+        </inertial>
         <visual>
             <origin xyz="0.0 0.0 -0.1125" rpy="0.0 0.0 0.0"/>
@@ -126,4 +229,13 @@
             </material>
         </visual>
+        <collision>
+            <origin xyz="0.0 0.0 -0.1125" rpy="0.0 0.0 0.0"/>
+            <geometry>
+                <mesh filename="package://mechabot_description/meshes/mechabot_toplid.stl" scale="0.001 0.001 0.001"/>
+            </geometry>
+            <material name="red">
+                <color rgba="0.6 0.0 0.0 1.0"/>
+            </material>
+        </collision>
     </link>
     <joint name="toplid_joint" type="fixed">

File: mechabot_ws/src/mechabot_description/urdf/mechabot_sensors.xacro (robot description, xacro)
@@ -2,4 +2,9 @@
 <robot name="mechabot" xmlns:xacro="http://www.ros.org/wiki/xacro">
     <link name="lidar_link">
+        <inertial>
+            <origin xyz="-0.028 0.0 -0.132" rpy="0.0 0.0 0.0"/>
+            <mass value="0.5"/>
+            <inertia ixx="0.1" ixy="0.0" ixz="0.0" iyy="0.1" iyz="0.0" izz="0.1"/>
+        </inertial>
         <visual>
             <origin xyz="-0.028 0.0 -0.132" rpy="0.0 0.0 0.0"/>
@@ -11,4 +16,13 @@
             </material>
         </visual>
+        <collision>
+            <origin xyz="-0.028 0.0 -0.132" rpy="0.0 0.0 0.0"/>
+            <geometry>
+                <mesh filename="package://mechabot_description/meshes/mechabot_lidar.stl" scale="0.001 0.001 0.001"/>
+            </geometry>
+            <material name="yellow">
+                <color rgba="0.6 0.6 0.0 1.0"/>
+            </material>
+        </collision>
     </link>
     <joint name="lidar_joint" type="fixed">
@@ -18,4 +32,9 @@
     </joint>
     <link name="camera_link">
+        <inertial>
+            <origin xyz="-0.118 0.0 -0.092" rpy="0.0 0.0 0.0"/>
+            <mass value="0.1"/>
+            <inertia ixx="0.1" ixy="0.0" ixz="0.0" iyy="0.1" iyz="0.0" izz="0.1"/>
+        </inertial>
         <visual>
             <origin xyz="-0.118 0.0 -0.092" rpy="0.0 0.0 0.0"/>
@@ -27,4 +46,13 @@
             </material>
         </visual>
+        <collision>
+            <origin xyz="-0.118 0.0 -0.092" rpy="0.0 0.0 0.0"/>
+            <geometry>
+                <mesh filename="package://mechabot_description/meshes/mechabot_camera.stl" scale="0.001 0.001 0.001"/>
+            </geometry>
+            <material name="green">
+                <color rgba="0.0 0.6 0.0 1.0"/>
+            </material>
+        </collision>
     </link>
     <joint name="camera_joint" type="fixed">
@@ -34,4 +62,9 @@
     </joint>
     <link name="imu_link">
+        <inertial>
+            <origin xyz="0.0 0.0 -0.035" rpy="0.0 0.0 0.0"/>
+            <mass value="0.1"/>
+            <inertia ixx="0.1" ixy="0.0" ixz="0.0" iyy="0.1" iyz="0.0" izz="0.1"/>
+        </inertial>
         <visual>
             <origin xyz="0.0 0.0 -0.035" rpy="0.0 0.0 0.0"/>
@@ -43,4 +76,13 @@
             </material>
         </visual>
+        <collision>
+            <origin xyz="0.0 0.0 -0.035" rpy="0.0 0.0 0.0"/>
+            <geometry>
+                <mesh filename="package://mechabot_description/meshes/mechabot_imu.stl" scale="0.001 0.001 0.001"/>
+            </geometry>
+            <material name="blue">
+                <color rgba="0.0 0.0 0.6 1.0"/>
+            </material>
+        </collision>
     </link>
     <joint name="imu_joint" type="fixed">
