Commit message: twist_mux added

File: mechabot_ws/src/mechabot_description/urdf/mechabot.urdf.xacro (robot description, xacro)
@@ -3,5 +3,5 @@
     <xacro:include filename="$(find mechabot_description)/urdf/mechabot_base.xacro" />
     <xacro:include filename="$(find mechabot_description)/urdf/mechabot_sensors.xacro"/>
-    <xacro:include filename="$(find mechabot_description)/urdf/gazebo.xacro"/>
-    <xacro:include filename="$(find mechabot_description)/urdf/ros2control.xacro"/>
+    <xacro:include filename="$(find mechabot_description)/urdf/mechabot_gazebo.xacro"/>
+    <xacro:include filename="$(find mechabot_description)/urdf/mechabot_ros2control.xacro"/>
 </robot>

File: mechabot_ws/src/mechabot_description/urdf/mechabot_base.xacro (robot description, xacro)
@@ -6,5 +6,5 @@
             <origin xyz="0.0 0.0 -0.0125" rpy="0.0 0.0 0.0"/>
             <mass value="5.0"/>
-            <inertia ixx="0.1" ixy="0.0" ixz="0.0" iyy="0.1" iyz="0.0" izz="0.1"/>
+            <inertia ixx="0.001" ixy="0.0" ixz="0.0" iyy="0.001" iyz="0.0" izz="0.001"/>
         </inertial>
         <visual>
@@ -36,5 +36,5 @@
             <origin xyz="0.0 0.0925 -0.034" rpy="0.0 0.0 0.0"/>
             <mass value="0.5"/>
-            <inertia ixx="0.1" ixy="0.0" ixz="0.0" iyy="0.1" iyz="0.0" izz="0.1"/>
+            <inertia ixx="0.001" ixy="0.0" ixz="0.0" iyy="0.001" iyz="0.0" izz="0.001"/>
         </inertial>
         <visual>
@@ -48,7 +48,8 @@
         </visual>
         <collision>
-            <origin xyz="0.0 0.0925 -0.034" rpy="0.0 0.0 0.0"/>
-            <geometry>
-                <mesh filename="package://mechabot_description/meshes/mechabot_right_wheel.stl" scale="0.001 0.001 0.001"/>
+            <origin xyz="0.0 0.0 -0.0" rpy="0.0 0.0 0.0"/>
+            <geometry>
+                <sphere radius="0.034"/>
+                <!-- <mesh filename="package://mechabot_description/meshes/mechabot_right_wheel.stl" scale="0.001 0.001 0.001"/> -->
             </geometry>
             <material name="blue">
@@ -67,5 +68,5 @@
             <origin xyz="0.0 -0.0925 -0.034" rpy="0.0 0.0 0.0"/>
             <mass value="0.5"/>
-            <inertia ixx="0.1" ixy="0.0" ixz="0.0" iyy="0.1" iyz="0.0" izz="0.1"/>
+            <inertia ixx="0.001" ixy="0.0" ixz="0.0" iyy="0.001" iyz="0.0" izz="0.001"/>
         </inertial>
         <visual>
@@ -79,7 +80,8 @@
         </visual>
         <collision>
-            <origin xyz="0.0 -0.0925 -0.034" rpy="0.0 0.0 0.0"/>
-            <geometry>
-                <mesh filename="package://mechabot_description/meshes/mechabot_left_wheel.stl" scale="0.001 0.001 0.001"/>
+            <origin xyz="0.0 0.0 -0.0" rpy="0.0 0.0 0.0"/>
+            <geometry>
+                <sphere radius="0.034"/>
+                <!-- <mesh filename="package://mechabot_description/meshes/mechabot_left_wheel.stl" scale="0.001 0.001 0.001"/> -->
             </geometry>
             <material name="blue">
@@ -98,5 +100,5 @@
             <origin xyz="-0.085 0.065 -0.021" rpy="0.0 0.0 0.0"/>
             <mass value="0.2"/>
-            <inertia ixx="0.1" ixy="0.0" ixz="0.0" iyy="0.1" iyz="0.0" izz="0.1"/>
+            <inertia ixx="0.001" ixy="0.0" ixz="0.0" iyy="0.001" iyz="0.0" izz="0.001"/>
         </inertial>
         <visual>
@@ -110,7 +112,8 @@
         </visual>
         <collision>
-            <origin xyz="-0.085 0.065 -0.021" rpy="0.0 0.0 0.0"/>
-            <geometry>
-                <mesh filename="package://mechabot_description/meshes/front_right_castor.stl" scale="0.001 0.001 0.001"/>
+            <origin xyz="0.0 0.0 -0.0125" rpy="0.0 0.0 0.0"/>
+            <geometry>
+                <sphere radius="0.00625"/>
+                <!-- <mesh filename="package://mechabot_description/meshes/front_right_castor.stl" scale="0.001 0.001 0.001"/> -->
             </geometry>
             <material name="grey">
@@ -120,5 +123,5 @@
     </link>
     <joint name="front_right_castor_joint" type="fixed">
-        <origin xyz="0.085 -0.065 0.0085" rpy="0.0 0.0 0.0"/>
+        <origin xyz="0.085 -0.065 0.00625" rpy="0.0 0.0 0.0"/>
         <parent link="base_link"/>
         <child link="front_right_castor_link"/>
@@ -128,5 +131,5 @@
             <origin xyz="-0.085 -0.065 -0.021" rpy="0.0 0.0 0.0"/>
             <mass value="0.2"/>
-            <inertia ixx="0.1" ixy="0.0" ixz="0.0" iyy="0.1" iyz="0.0" izz="0.1"/>
+            <inertia ixx="0.001" ixy="0.0" ixz="0.0" iyy="0.001" iyz="0.0" izz="0.001"/>
         </inertial>
         <visual>
@@ -140,7 +143,8 @@
         </visual>
         <collision>
-            <origin xyz="-0.085 -0.065 -0.021" rpy="0.0 0.0 0.0"/>
-            <geometry>
-                <mesh filename="package://mechabot_description/meshes/front_left_castor.stl" scale="0.001 0.001 0.001"/>
+            <origin xyz="0.0 0.0 -0.0125" rpy="0.0 0.0 0.0"/>
+            <geometry>
+                <sphere radius="0.00625"/>
+                <!-- <mesh filename="package://mechabot_description/meshes/front_left_castor.stl" scale="0.001 0.001 0.001"/> -->
             </geometry>
             <material name="grey">
@@ -150,5 +154,5 @@
     </link>
     <joint name="front_left_castor_joint" type="fixed">
-        <origin xyz="0.085 0.065 0.0085" rpy="0.0 0.0 0.0"/>
+        <origin xyz="0.085 0.065 0.00625" rpy="0.0 0.0 0.0"/>
         <parent link="base_link"/>
         <child link="front_left_castor_link"/>
@@ -158,5 +162,5 @@
             <origin xyz="0.085 0.065 -0.0205" rpy="0.0 0.0 0.0"/>
             <mass value="0.2"/>
-            <inertia ixx="0.1" ixy="0.0" ixz="0.0" iyy="0.1" iyz="0.0" izz="0.1"/>
+            <inertia ixx="0.001" ixy="0.0" ixz="0.0" iyy="0.001" iyz="0.0" izz="0.001"/>
         </inertial>
         <visual>
@@ -170,7 +174,8 @@
         </visual>
         <collision>
-            <origin xyz="0.085 0.065 -0.0205" rpy="0.0 0.0 0.0"/>
-            <geometry>
-                <mesh filename="package://mechabot_description/meshes/rear_right_castor.stl" scale="0.001 0.001 0.001"/>
+            <origin xyz="0.0 0.0 -0.0125" rpy="0.0 0.0 0.0"/>
+            <geometry>
+                <sphere radius="0.00625"/>
+                <!-- <mesh filename="package://mechabot_description/meshes/rear_right_castor.stl" scale="0.001 0.001 0.001"/> -->
             </geometry>
             <material name="grey">
@@ -180,5 +185,5 @@
     </link>
     <joint name="rear_right_castor_joint" type="fixed">
-        <origin xyz="-0.085 -0.065 0.008" rpy="0.0 0.0 0.0"/>
+        <origin xyz="-0.085 -0.065 0.00635" rpy="0.0 0.0 0.0"/>
         <parent link="base_link"/>
         <child link="rear_right_castor_link"/>
@@ -188,5 +193,5 @@
             <origin xyz="0.085 -0.065 -0.0205" rpy="0.0 0.0 0.0"/>
             <mass value="0.2"/>
-            <inertia ixx="0.1" ixy="0.0" ixz="0.0" iyy="0.1" iyz="0.0" izz="0.1"/>
+            <inertia ixx="0.001" ixy="0.0" ixz="0.0" iyy="0.001" iyz="0.0" izz="0.001"/>
         </inertial>
         <visual>
@@ -200,7 +205,8 @@
         </visual>
         <collision>
-            <origin xyz="0.085 -0.065 -0.0205" rpy="0.0 0.0 0.0"/>
-            <geometry>
-                <mesh filename="package://mechabot_description/meshes/rear_left_castor.stl" scale="0.001 0.001 0.001"/>
+            <origin xyz="0.0 0.0 -0.0125" rpy="0.0 0.0 0.0"/>
+            <geometry>
+                <sphere radius="0.00625"/>
+                <!-- <mesh filename="package://mechabot_description/meshes/rear_left_castor.stl" scale="0.001 0.001 0.001"/> -->
             </geometry>
             <material name="grey">
@@ -210,5 +216,5 @@
     </link>
     <joint name="rear_left_castor_joint" type="fixed">
-        <origin xyz="-0.085 0.065 0.008" rpy="0.0 0.0 0.0"/>
+        <origin xyz="-0.085 0.065 0.00635" rpy="0.0 0.0 0.0"/>
         <parent link="base_link"/>
         <child link="rear_left_castor_link"/>
@@ -216,7 +222,7 @@
     <link name="toplid_link">
         <inertial>
-            <origin xyz="0.0 0.0 -0.1125" rpy="0.0 0.0 0.0"/>
+            <origin xyz="0.0 0.0 -0.001125" rpy="0.0 0.0 0.0"/>
             <mass value="2.0"/>
-            <inertia ixx="0.1" ixy="0.0" ixz="0.0" iyy="0.1" iyz="0.0" izz="0.1"/>
+            <inertia ixx="0.001" ixy="0.0" ixz="0.0" iyy="0.001" iyz="0.0" izz="0.001"/>
         </inertial>
         <visual>

File: mechabot_ws/src/mechabot_description/urdf/mechabot_gazebo.xacro (robot description, xacro)
@@ -22,6 +22,6 @@
     <!-- Caster Wheels -->
     <gazebo reference="front_right_castor_link">
-        <mu1>0.1</mu1>
-        <mu2>0.1</mu2>
+        <mu1>0.01</mu1>
+        <mu2>0.01</mu2>
         <kp>1000000.0</kp>
         <kd>100.0</kd>
@@ -30,6 +30,6 @@
     </gazebo>
     <gazebo reference="front_left_castor_link">
-        <mu1>0.1</mu1>
-        <mu2>0.1</mu2>
+        <mu1>0.01</mu1>
+        <mu2>0.01</mu2>
         <kp>1000000.0</kp>
         <kd>100.0</kd>
@@ -38,6 +38,6 @@
     </gazebo>
     <gazebo reference="rear_right_castor_link">
-        <mu1>0.1</mu1>
-        <mu2>0.1</mu2>
+        <mu1>0.01</mu1>
+        <mu2>0.01</mu2>
         <kp>1000000.0</kp>
         <kd>100.0</kd>
@@ -46,6 +46,6 @@
     </gazebo>
     <gazebo reference="rear_left_castor_link">
-        <mu1>0.1</mu1>
-        <mu2>0.1</mu2>
+        <mu1>0.01</mu1>
+        <mu2>0.01</mu2>
         <kp>1000000.0</kp>
         <kd>100.0</kd>
@@ -58,4 +58,38 @@
             <parameters>$(find mechabot_controller)/config/mechabot_controllers.yaml</parameters>
         </plugin>
+        <plugin filename="ignition-gazebo-sensors-system" name="ignition::gazebo::systems::Sensors">
+            <render_engine>ogre2</render_engine>
+        </plugin>
+    </gazebo>
+    <!-- MechaBot Sensors-->
+    <gazebo reference="lidar_link">
+        <sensor name="lidar" type="gpu_lidar">
+            <pose>0 0 0 0 0 0</pose>
+            <always_on>true</always_on>
+            <visualize>true</visualize>
+            <topic>scan</topic>
+            <update_rate>5</update_rate>
+            <gz_frame_id>lidar_link</gz_frame_id>
+            <lidar>
+                <scan>
+                    <horizontal>
+                        <samples>360</samples>
+                        <resolution>1.00000</resolution>
+                        <min_angle>0.000000</min_angle>
+                        <max_angle>6.280000</max_angle>
+                    </horizontal>
+                </scan>
+                <range>
+                    <min>0.15</min>
+                    <max>12.0</max>
+                    <resolution>0.02</resolution>
+                </range>
+                <noise>
+                    <type>gaussian</type>
+                    <mean>0.0</mean>
+                    <stddev>0.01</stddev>
+                </noise>
+            </lidar>
+        </sensor>
     </gazebo>
 </robot>

File: mechabot_ws/src/mechabot_description/urdf/mechabot_ros2control.xacro (robot description, xacro)
@@ -7,6 +7,6 @@
         <joint name="right_wheel_joint">
             <command_interface name="velocity">
-                <param name="min">-4.5</param>
-                <param name="max">4.5</param>
+                <param name="min">-2.0</param>
+                <param name="max">2.0</param>
             </command_interface>
             <state_interface name="position" />
@@ -15,6 +15,6 @@
         <joint name="left_wheel_joint">
             <command_interface name="velocity">
-                <param name="min">-4.5</param>
-                <param name="max">4.5</param>
+                <param name="min">-2.0</param>
+                <param name="max">2.0</param>
             </command_interface>
             <state_interface name="position" />

File: mechabot_ws/src/mechabot_description/urdf/mechabot_sensors.xacro (robot description, xacro)
@@ -5,5 +5,5 @@
             <origin xyz="-0.028 0.0 -0.132" rpy="0.0 0.0 0.0"/>
             <mass value="0.5"/>
-            <inertia ixx="0.1" ixy="0.0" ixz="0.0" iyy="0.1" iyz="0.0" izz="0.1"/>
+            <inertia ixx="0.001" ixy="0.0" ixz="0.0" iyy="0.001" iyz="0.0" izz="0.001"/>
         </inertial>
         <visual>
@@ -35,5 +35,5 @@
             <origin xyz="-0.118 0.0 -0.092" rpy="0.0 0.0 0.0"/>
             <mass value="0.1"/>
-            <inertia ixx="0.1" ixy="0.0" ixz="0.0" iyy="0.1" iyz="0.0" izz="0.1"/>
+            <inertia ixx="0.001" ixy="0.0" ixz="0.0" iyy="0.001" iyz="0.0" izz="0.001"/>
         </inertial>
         <visual>
@@ -65,5 +65,5 @@
             <origin xyz="0.0 0.0 -0.035" rpy="0.0 0.0 0.0"/>
             <mass value="0.1"/>
-            <inertia ixx="0.1" ixy="0.0" ixz="0.0" iyy="0.1" iyz="0.0" izz="0.1"/>
+            <inertia ixx="0.001" ixy="0.0" ixz="0.0" iyy="0.001" iyz="0.0" izz="0.001"/>
         </inertial>
         <visual>
